File: metallali_pcb/metallali.kicad_pcb (KiCad board)
At the start: 2 copper layers, 317.9 x 132.8 mm, 110 parts, among them J2 USB_C_Receptacle_USB2.0_14P, SW1 SW_DPST_x2, SW2 SW_DPST_x2, U1 STM32F072CBTx, U2 XC6206PxxxMR, U3 SRV05-4

Commit message: Routed matrix
Parts:
- moved F1 52.4 mm to (206.2, 56.1), turned to -90 degrees
- moved U3 38.4 mm to (202.9, 63.5), turned to 90 degrees
- moved U2 30.7 mm to (202.9, 70.8), turned to 90 degrees
- moved SW2 14.0 mm to (215.2, 92.1)
- moved SW1 12.1 mm to (212.5, 82.2)
- moved R3 5.63 mm to (204.5, 54.4), turned to -90 degrees
- moved R2 5.50 mm to (201.5, 54.3), turned to -90 degrees
Routing:
- net ROW5: track 117.3 -> 173.0 mm
- net ROW7: track 129.1 -> 181.8 mm
- net ROW0: track 108.9 -> 160.7 mm
- net ROW2: track 114.5 -> 166.0 mm
- net ROW6: track 121.0 -> 171.9 mm
- net ROW1: track 116.9 -> 166.2 mm
- net ROW4: track 114.8 -> 162.9 mm
- net ROW3: track 132.5 -> 171.3 mm
- net +5V: track 0.00 -> 17.4 mm, vias 0 -> 4
- net DP: track 0.00 -> 14.1 mm
- net DN: track 0.00 -> 13.4 mm
- net VBUS: track 0.00 -> 10.7 mm
- net COL3: track 95.8 -> 101.5 mm
- net COL11: track 98.6 -> 103.2 mm
- net COL8: track 95.9 -> 100.5 mm
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
Commit message: Almost done! Just need to draw the outline of the PCB.
Parts:
- added H1: MountingHole_Pad, MountingHole:MountingHole_3.2mm_M3_ISO14580_Pad, F.Cu at (202.6, 135.0)
- added H2: MountingHole_Pad, MountingHole:MountingHole_3.2mm_M3_ISO14580_Pad, F.Cu at (223.0, 47.0)
- added H3: MountingHole_Pad, MountingHole:MountingHole_3.2mm_M3_ISO14580_Pad, F.Cu at (333.5, 30.5)
- added H4: MountingHole_Pad, MountingHole:MountingHole_3.2mm_M3_ISO14580_Pad, F.Cu at (360.0, 124.0)
- added H5: MountingHole_Pad, MountingHole:MountingHole_3.2mm_M3_ISO14580_Pad, F.Cu at (296.0, 113.0)
- added H6: MountingHole_Pad, MountingHole:MountingHole_3.2mm_M3_ISO14580_Pad, F.Cu at (182.2, 47.0)
- added H7: MountingHole_Pad, MountingHole:MountingHole_3.2mm_M3_ISO14580_Pad, F.Cu at (71.7, 30.1)
- added H8: MountingHole_Pad, MountingHole:MountingHole_3.2mm_M3_ISO14580_Pad, F.Cu at (45.2, 124.0)
- added H9: MountingHole_Pad, MountingHole:MountingHole_3.2mm_M3_ISO14580_Pad, F.Cu at (109.2, 113.0)
- D1, D10, D11, D12, D13, D14, D15, D16, D17, D18, D19, D2, D20, D21, D22, D23, D24, D25, D26, D27, D28, D29, D3, D30, D31, D32, D33, D34, D35, D36, D37, D38, D39, D4, D40, D41, D42, D43, D44, D45, D46, D5, D6, D7, D8, D9: footprint Diode_SMD:D_SOD-123 -> Diode_SMD:D_SOD-323
- moved C1 38.1 mm to (205.5, 120.0), turned to -90 degrees
- moved SW1 35.8 mm to (197.8, 114.8), turned to -90 degrees
- moved U1 32.6 mm to (202.6, 84.8), turned to 45 degrees
- moved C7 29.6 mm to (202.6, 67.0), turned to 180 degrees
- moved C8 25.6 mm to (202.6, 73.2), turned to 180 degrees
- moved R1 24.1 mm to (199.7, 120.0), turned to -90 degrees
- moved SW2 24.0 mm to (207.3, 114.8), turned to 90 degrees
- moved C5 17.0 mm to (204.6, 78.0), turned to 45 degrees
- moved C3 14.9 mm to (209.2, 86.9), turned to -45 degrees
- moved C6 5.94 mm to (199.4, 90.5), turned to -135 degrees
- moved C2 3.67 mm to (196.2, 82.5), turned to 135 degrees
- moved C4 3.02 mm to (196.2, 87.2), turned to -135 degrees
- moved F1 0.90 mm to (207.0, 55.8)
- moved U2 0.89 mm to (202.6, 70.0)
- moved J2 0.66 mm to (202.6, 47.4)
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Connections:
- U1 pad 19: unconnected-(U1-PB1-Pad19) -> ROW7
- U1 pad 20: unconnected-(U1-PB2-Pad20) -> COL11
- U1 pad 21: unconnected-(U1-PB10-Pad21) -> COL10
- U1 pad 25: unconnected-(U1-PB12-Pad25) -> COL9
- U1 pad 26: unconnected-(U1-PB13-Pad26) -> COL8
- U1 pad 27: unconnected-(U1-PB14-Pad27) -> COL7
- U1 pad 28: unconnected-(U1-PB15-Pad28) -> COL6
- U1 pad 29: unconnected-(U1-PA8-Pad29) -> ROW6
- U1 pad 3: unconnected-(U1-PC14-Pad3) -> COL1
- U1 pad 30: unconnected-(U1-PA9-Pad30) -> ROW5
- U1 pad 31: unconnected-(U1-PA10-Pad31) -> ROW4
- U1 pad 37: unconnected-(U1-PA14-Pad37) -> ROW0
- U1 pad 38: unconnected-(U1-PA15-Pad38) -> ROW1
- U1 pad 39: unconnected-(U1-PB3-Pad39) -> ROW2
- U1 pad 4: unconnected-(U1-PC15-Pad4) -> COL0
- U1 pad 40: unconnected-(U1-PB4-Pad40) -> COL5
- U1 pad 41: unconnected-(U1-PB5-Pad41) -> COL4
- U1 pad 42: unconnected-(U1-PB6-Pad42) -> COL3
- U1 pad 43: unconnected-(U1-PB7-Pad43) -> COL2
- U1 pad 5: unconnected-(U1-PF0-Pad5) -> ROW3
Routing:
- net COL11: track 103.2 -> 261.2 mm
- net COL0: track 101.3 -> 258.9 mm
- net COL1: track 102.1 -> 238.1 mm
- net COL10: track 102.5 -> 237.4 mm
- net COL2: track 54.1 -> 177.9 mm
- net COL9: track 54.1 -> 175.4 mm
- net COL3: track 101.5 -> 208.3 mm
- net COL8: track 100.5 -> 205.0 mm
- net COL4: track 99.5 -> 184.3 mm
- net COL7: track 99.6 -> 182.0 mm
- net +3V3: track 0.00 -> 78.4 mm, vias 0 -> 2
- net COL5: track 102.5 -> 165.8 mm
- net COL6: track 103.1 -> 161.7 mm
- net BOOT-1: track 0.00 -> 42.4 mm, vias 0 -> 2
- net ROW3: track 171.3 -> 209.1 mm
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- added copper zone on B.Cu, net GND
- added copper zone on F.Cu, net GND
Other:
- board size 317.9 x 132.8 mm -> 349.6 x 146.9 mm
- board text added: "Boot"
- board text added: "Reset"

Commit message: Finished v1.0.00 pcb
Parts:
- added H10: MountingHole_Pad, MountingHole:MountingHole_3.2mm_M3_ISO14580_Pad, F.Cu at (30.2, 112.8)
- added H11: MountingHole_Pad, MountingHole:MountingHole_3.2mm_M3_ISO14580_Pad, F.Cu at (95.2, 143.2)
- added H12: MountingHole_Pad, MountingHole:MountingHole_3.2mm_M3_ISO14580_Pad, F.Cu at (179.0, 163.7)
- moved H8 131.2 mm to (133.4, 26.9)
- moved H6 124.7 mm to (226.2, 163.7)
- moved H7 108.8 mm to (179.3, 46.0)
- moved H1 92.0 mm to (225.9, 46.0)
- moved H9 90.6 mm to (67.2, 32.7)
- moved H2 52.7 mm to (271.8, 26.9)
- moved H5 33.2 mm to (310.0, 143.2)
- moved H4 18.7 mm to (374.9, 112.8)
- moved H3 4.99 mm to (338.0, 32.7)
- moved F1 2.36 mm to (207.0, 53.4)
- moved J2 2.36 mm to (202.6, 45.1)
- moved R2 2.36 mm to (201.0, 51.6)
- moved R3 2.36 mm to (204.2, 51.6)
Routing:
- net +5V: track 17.4 -> 19.8 mm
- net DP: track 37.6 -> 40.0 mm
- net DN: track 36.5 -> 38.8 mm
Other:
- board size 349.6 x 146.9 mm -> 355.7 x 151.5 mm
- board text added: "Designed by My-Fi"
