File: metallali_pcb/metallali.kicad_sch (KiCad schematic)
At the start: 110 parts, among them J2 USB_C_Receptacle_USB2.0_14P, SW1 SW_DPST_x2, SW2 SW_DPST_x2, U1 STM32F072CBTx, U2 XC6206PxxxMR, U3 SRV05-4

Commit message: Almost done! Just need to draw the outline of the PCB.
Parts:
- added H1, H2, H3, H4, H5, H6, H7, H8, H9: MountingHole_Pad, MountingHole:MountingHole_3.2mm_M3_ISO14580_Pad, symbol Mechanical:MountingHole_Pad
- D1, D10, D11, D12, D13, D14, D15, D16, D17, D18, D19, D2, D20, D21, D22, D23, D24, D25, D26, D27, D28, D29, D3, D30, D31, D32, D33, D34, D35, D36, D37, D38, D39, D4, D40, D41, D42, D43, D44, D45, D46, D5, D6, D7, D8, D9: footprint Diode_SMD:D_SOD-123 -> Diode_SMD:D_SOD-323
Connections:
- net COL0: now also U1.4 (PC15)
- net COL1: now also U1.3 (PC14)
- net COL10: now also U1.21 (PB10)
- net COL11: now also U1.20 (PB2)
- net COL2: now also U1.43 (PB7)
- net COL3: now also U1.42 (PB6)
- net COL4: now also U1.41 (PB5)
- net COL5: now also U1.40 (PB4)
- net COL6: now also U1.28 (PB15)
- net COL7: now also U1.27 (PB14)
- net COL8: now also U1.26 (PB13)
- net COL9: now also U1.25 (PB12)
- net GND: now also H1.1, H2.1, H3.1, H4.1, H5.1, H6.1, H7.1, H8.1, H9.1
- net ROW0: now also U1.37 (PA14)
- net ROW1: now also U1.38 (PA15)
- net ROW2: now also U1.39 (PB3)
- net ROW3: now also U1.5 (PF0)
- net ROW4: now also U1.31 (PA10)
- net ROW5: now also U1.30 (PA9)
- net ROW6: now also U1.29 (PA8)
- net ROW7: now also U1.19 (PB1)
- no-connect marks 5 -> 17

Commit message: Finished v1.0.00 pcb
Parts:
- added H10, H11, H12: MountingHole_Pad, MountingHole:MountingHole_3.2mm_M3_ISO14580_Pad, symbol Mechanical:MountingHole_Pad
Connections:
- net GND: now also H10.1, H11.1, H12.1
